Commit message: Dosya isimleri ve hatalar duzeltildi

File: description/robot_core.xacro (robot description, xacro)
@@ -1,4 +1,5 @@
 <?xml version="1.0"?>
 <robot xmlns:xacro="http://www.ros.org/wiki/xacro" >
+<xacro:include filename="inertial_macros.xacro"/>
 <material name="white">
     <color rgba="1 1 1 1"/>
@@ -35,4 +36,7 @@
         </geometry>
     </collision>
+    <xacro:inertial_box mass="0.5" x="0.3" y="0.3" z="0.15">
+        <origin xyz="0.15 0 0.075" rpy="0 0 0"/>
+    </xacro:inertial_box>
 </link>
 <!-- SOL TEKERLEK ÇİZİMİ -->
@@ -55,4 +59,7 @@
         </geometry>
     </collision>
+    <xacro:inertial_cylinder mass="0.1" length="0.04" radius="0.05">
+        <origin xyz="0 0 0" rpy="0 0 0"/>
+    </xacro:inertial_cylinder>
 </link>
 <!-- SAĞ TEKERLEK ÇİZİMİ -->
@@ -75,4 +82,7 @@
         </geometry>
     </collision>
+    <xacro:inertial_cylinder mass="0.1" length="0.04" radius="0.05">
+        <origin xyz="0 0 0" rpy="0 0 0"/>
+    </xacro:inertial_cylinder>
 </link>
 <!-- ÖN TEKERLEK ÇİZİMİ -->
@@ -94,4 +104,7 @@
         </geometry>
     </collision>
+    <xacro:inertial_sphere mass="0.1" radius="0.05">
+        <origin xyz="0 0 0" rpy="0 0 0"/>
+    </xacro:inertial_sphere>
 </link>
 </robot>
